File: Hardware/common/common.brd (EAGLE design)
At the start: 81.3 x 81.3 mm, 24 parts, among them U1 788BS, U10 788BS, U11 788BS, U12 788BS, U13 788BS, U14 788BS, U15 788BS, U16 788BS, U2 788BS, U3 788BS, U4 788BS, U5 788BS, U6 788BS, U7 788BS, U8 788BS, U9 788BS

Commit message: Got row/col reversed
Parts:
- removed U1, U10, U11, U12, U13, U14, U15, U16, U2, U3, U4, U5, U6, U7, U8, U9: 788BS, ledmatrix:788BS8X81.9MM
- added U$1, U$10, U$11, U$12, U$13, U$14, U$15, U$16, U$2, U$3, U$4, U$5, U$6, U$7, U$8, U$9: 788BS-V2, ledmatrix-v2:788BS8X81.9MM-V2
Connections:
- net COL1: now also U$1.P5, U$13.P5, U$5.P5, U$9.P5; no longer U1.P13, U13.P13, U4.P13, U7.P13
- net COL10: now also U$10.P2, U$14.P2, U$2.P2, U$6.P2; no longer U14.P3, U2.P3, U5.P3, U8.P3
- net COL11: now also U$10.P7, U$14.P7, U$2.P7, U$6.P7; no longer U14.P4, U2.P4, U5.P4, U8.P4
- net COL12: now also U$10.P1, U$14.P1, U$2.P1, U$6.P1; no longer U14.P10, U2.P10, U5.P10, U8.P10
- net COL13: now also U$10.P12, U$14.P12, U$2.P12, U$6.P12; no longer U14.P6, U2.P6, U5.P6, U8.P6
- net COL14: now also U$10.P8, U$14.P8, U$2.P8, U$6.P8; no longer U14.P11, U2.P11, U5.P11, U8.P11
- net COL15: now also U$10.P14, U$14.P14, U$2.P14, U$6.P14; no longer U14.P15, U2.P15, U5.P15, U8.P15
- net COL16: now also U$10.P9, U$14.P9, U$2.P9, U$6.P9; no longer U14.P16, U2.P16, U5.P16, U8.P16
- net COL17: now also U$11.P5, U$15.P5, U$3.P5, U$7.P5; no longer U15.P13, U3.P13, U6.P13, U9.P13
- net COL18: now also U$11.P2, U$15.P2, U$3.P2, U$7.P2; no longer U15.P3, U3.P3, U6.P3, U9.P3
- net COL19: now also U$11.P7, U$15.P7, U$3.P7, U$7.P7; no longer U15.P4, U3.P4, U6.P4, U9.P4
- net COL2: now also U$1.P2, U$13.P2, U$5.P2, U$9.P2; no longer U1.P3, U13.P3, U4.P3, U7.P3
- net COL20: now also U$11.P1, U$15.P1, U$3.P1, U$7.P1; no longer U15.P10, U3.P10, U6.P10, U9.P10
- net COL21: now also U$11.P12, U$15.P12, U$3.P12, U$7.P12; no longer U15.P6, U3.P6, U6.P6, U9.P6
- net COL22: now also U$11.P8, U$15.P8, U$3.P8, U$7.P8; no longer U15.P11, U3.P11, U6.P11, U9.P11
- net COL23: now also U$11.P14, U$15.P14, U$3.P14, U$7.P14; no longer U15.P15, U3.P15, U6.P15, U9.P15
- net COL24: now also U$11.P9, U$15.P9, U$3.P9, U$7.P9; no longer U15.P16, U3.P16, U6.P16, U9.P16
- net COL25: now also U$12.P5, U$16.P5, U$4.P5, U$8.P5; no longer U10.P13, U11.P13, U12.P13, U16.P13
- net COL26: now also U$12.P2, U$16.P2, U$4.P2, U$8.P2; no longer U10.P3, U11.P3, U12.P3, U16.P3
- net COL27: now also U$12.P7, U$16.P7, U$4.P7, U$8.P7; no longer U10.P4, U11.P4, U12.P4, U16.P4
- net COL28: now also U$12.P1, U$16.P1, U$4.P1, U$8.P1; no longer U10.P10, U11.P10, U12.P10, U16.P10
- net COL29: now also U$12.P12, U$16.P12, U$4.P12, U$8.P12; no longer U10.P6, U11.P6, U12.P6, U16.P6
- net COL3: now also U$1.P7, U$13.P7, U$5.P7, U$9.P7; no longer U1.P4, U13.P4, U4.P4, U7.P4
- net COL30: now also U$12.P8, U$16.P8, U$4.P8, U$8.P8; no longer U10.P11, U11.P11, U12.P11, U16.P11
- net COL31: now also U$12.P14, U$16.P14, U$4.P14, U$8.P14; no longer U10.P15, U11.P15, U12.P15, U16.P15
- net COL32: now also U$12.P9, U$16.P9, U$4.P9, U$8.P9; no longer U10.P16, U11.P16, U12.P16, U16.P16
- net COL4: now also U$1.P1, U$13.P1, U$5.P1, U$9.P1; no longer U1.P10, U13.P10, U4.P10, U7.P10
- net COL5: now also U$1.P12, U$13.P12, U$5.P12, U$9.P12; no longer U1.P6, U13.P6, U4.P6, U7.P6
- net COL6: now also U$1.P8, U$13.P8, U$5.P8, U$9.P8; no longer U1.P11, U13.P11, U4.P11, U7.P11
- net COL7: now also U$1.P14, U$13.P14, U$5.P14, U$9.P14; no longer U1.P15, U13.P15, U4.P15, U7.P15
- net COL8: now also U$1.P9, U$13.P9, U$5.P9, U$9.P9; no longer U1.P16, U13.P16, U4.P16, U7.P16
- net COL9: now also U$10.P5, U$14.P5, U$2.P5, U$6.P5; no longer U14.P13, U2.P13, U5.P13, U8.P13
- net ROW1: now also U$1.P13, U$2.P13, U$3.P13, U$4.P13; no longer U1.P9, U10.P9, U2.P9, U3.P9
- net ROW10: now also U$5.P3, U$6.P3, U$7.P3, U$8.P3; no longer U11.P14, U4.P14, U5.P14, U6.P14
- net ROW11: now also U$5.P4, U$6.P4, U$7.P4, U$8.P4; no longer U11.P8, U4.P8, U5.P8, U6.P8
- net ROW12: now also U$5.P10, U$6.P10, U$7.P10, U$8.P10; no longer U11.P12, U4.P12, U5.P12, U6.P12
- net ROW13: now also U$5.P6, U$6.P6, U$7.P6, U$8.P6; no longer U11.P1, U4.P1, U5.P1, U6.P1
- net ROW14: now also U$5.P11, U$6.P11, U$7.P11, U$8.P11; no longer U11.P7, U4.P7, U5.P7, U6.P7
- net ROW15: now also U$5.P15, U$6.P15, U$7.P15, U$8.P15; no longer U11.P2, U4.P2, U5.P2, U6.P2
- net ROW16: now also U$5.P16, U$6.P16, U$7.P16, U$8.P16; no longer U11.P5, U4.P5, U5.P5, U6.P5
- net ROW17: now also U$10.P13, U$11.P13, U$12.P13, U$9.P13; no longer U12.P9, U7.P9, U8.P9, U9.P9
- net ROW18: now also U$10.P3, U$11.P3, U$12.P3, U$9.P3; no longer U12.P14, U7.P14, U8.P14, U9.P14
- net ROW19: now also U$10.P4, U$11.P4, U$12.P4, U$9.P4; no longer U12.P8, U7.P8, U8.P8, U9.P8
- net ROW2: now also U$1.P3, U$2.P3, U$3.P3, U$4.P3; no longer U1.P14, U10.P14, U2.P14, U3.P14
- net ROW20: now also U$10.P10, U$11.P10, U$12.P10, U$9.P10; no longer U12.P12, U7.P12, U8.P12, U9.P12
- net ROW21: now also U$10.P6, U$11.P6, U$12.P6, U$9.P6; no longer U12.P1, U7.P1, U8.P1, U9.P1
- net ROW22: now also U$10.P11, U$11.P11, U$12.P11, U$9.P11; no longer U12.P7, U7.P7, U8.P7, U9.P7
- net ROW23: now also U$10.P15, U$11.P15, U$12.P15, U$9.P15; no longer U12.P2, U7.P2, U8.P2, U9.P2
- net ROW24: now also U$10.P16, U$11.P16, U$12.P16, U$9.P16; no longer U12.P5, U7.P5, U8.P5, U9.P5
- net ROW25: now also U$13.P13, U$14.P13, U$15.P13, U$16.P13; no longer U13.P9, U14.P9, U15.P9, U16.P9
- net ROW26: now also U$13.P3, U$14.P3, U$15.P3, U$16.P3; no longer U13.P14, U14.P14, U15.P14, U16.P14
- net ROW27: now also U$13.P4, U$14.P4, U$15.P4, U$16.P4; no longer U13.P8, U14.P8, U15.P8, U16.P8
- net ROW28: now also U$13.P10, U$14.P10, U$15.P10, U$16.P10; no longer U13.P12, U14.P12, U15.P12, U16.P12
- net ROW29: now also U$13.P6, U$14.P6, U$15.P6, U$16.P6; no longer U13.P1, U14.P1, U15.P1, U16.P1
- net ROW3: now also U$1.P4, U$2.P4, U$3.P4, U$4.P4; no longer U1.P8, U10.P8, U2.P8, U3.P8
- net ROW30: now also U$13.P11, U$14.P11, U$15.P11, U$16.P11; no longer U13.P7, U14.P7, U15.P7, U16.P7
- net ROW31: now also U$13.P15, U$14.P15, U$15.P15, U$16.P15; no longer U13.P2, U14.P2, U15.P2, U16.P2
- net ROW32: now also U$13.P16, U$14.P16, U$15.P16, U$16.P16; no longer U13.P5, U14.P5, U15.P5, U16.P5
- net ROW4: now also U$1.P10, U$2.P10, U$3.P10, U$4.P10; no longer U1.P12, U10.P12, U2.P12, U3.P12
- net ROW5: now also U$1.P6, U$2.P6, U$3.P6, U$4.P6; no longer U1.P1, U10.P1, U2.P1, U3.P1
- net ROW6: now also U$1.P11, U$2.P11, U$3.P11, U$4.P11; no longer U1.P7, U10.P7, U2.P7, U3.P7
- net ROW7: now also U$1.P15, U$2.P15, U$3.P15, U$4.P15; no longer U1.P2, U10.P2, U2.P2, U3.P2
- net ROW8: now also U$1.P16, U$2.P16, U$3.P16, U$4.P16; no longer U1.P5, U10.P5, U2.P5, U3.P5
- net ROW9: now also U$5.P13, U$6.P13, U$7.P13, U$8.P13; no longer U11.P9, U4.P9, U5.P9, U6.P9
Routing:
- net ROW12: track 67.7 -> 176.5 mm, vias 1 -> 6
- net COL7: track 239.0 -> 136.0 mm, vias 8 -> 9
- net COL3: track 176.3 -> 276.3 mm, vias 3 -> 7
- net ROW11: track 85.6 -> 170.2 mm, vias 1 -> 5
- net ROW9: track 183.5 -> 107.2 mm, vias 6 -> 5
- net COL20: track 148.0 -> 91.5 mm, vias 4 -> 5
- net COL13: track 135.6 -> 83.2 mm, vias 5 -> 0
- net COL32: track 113.4 -> 72.3 mm, vias 1 -> 0
- net COL9: track 80.6 -> 120.2 mm, vias 1 -> 6
- net COL12: track 98.8 -> 138.2 mm, vias 4 -> 8
- net COL4: track 204.5 -> 166.2 mm, vias 6 -> 5
- net COL23: track 105.0 -> 69.4 mm, vias 3 -> 2
- net ROW17: track 86.1 -> 121.7 mm, vias 1 -> 8
- net ROW22: track 139.5 -> 107.9 mm, vias 2 -> 5
- net ROW32: track 74.1 -> 100.6 mm
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Other:
- outline, holes or cut-outs redrawn
- board text added: "LED 32x32 Matrix Display Breakout RevB"
- board text added: "ROWXX: CATHODE COLXX: ANODE"
- board text removed: "LED 32x32 Matrix Display Breakout RevA"
- board text removed: "ROWXX: ANODE COLXX: CATHODE"
