File: Hardware/py32f030f18p6/py32f030f18p6-led.sch (EAGLE design)
At the start: 132 parts, among them IC2 AP2114HA-3.3TRG1, J10 455-1750-1-ND, J11 455-1750-1-ND, J12 455-1750-1-ND, J14 USB_MINI-B_SMT, J15 455-1750-1-ND, J16 455-1750-1-ND, J9 455-1750-1-ND, Q1 MMBT3904LT3G, Q10 MMBT3904LT3G, Q11 MMBT3904LT3G, Q12 MMBT3904LT3G, Q13 MMBT3904LT3G, Q14 MMBT3904LT3G, Q15 MMBT3904LT3G, Q16 MMBT3904LT3G, Q17 MMBT3904LT3G, Q18 MMBT3904LT3G, Q19 MMBT3904LT3G, Q2 MMBT3904LT3G, Q20 MMBT3904LT3G, Q21 MMBT3904LT3G, Q22 MMBT3904LT3G, Q23 MMBT3904LT3G, Q24 MMBT3904LT3G, Q25 MMBT3904LT3G, Q26 MMBT3904LT3G, Q27 MMBT3904LT3G, Q28 MMBT3904LT3G, Q29 MMBT3904LT3G, Q3 MMBT3904LT3G, Q30 MMBT3904LT3G, Q31 MMBT3904LT3G, Q32 MMBT3904LT3G, Q4 MMBT3904LT3G, Q5 MMBT3904LT3G, Q6 MMBT3904LT3G, Q7 MMBT3904LT3G, Q8 MMBT3904LT3G, Q9 MMBT3904LT3G, U1 TC74HC595AF(EL,F), U2 TC74HC595AF(EL,F), U3 TC74HC595AF(EL,F), U4 TC74HC595AF(EL,F), U5 TC74HC595AF(EL,F), U6 TC74HC595AF(EL,F), U7 TC74HC595AF(EL,F), U8 TC74HC595AF(EL,F)

Commit message: Got row/col reversed
Parts:
- renumbered J1 to J1ROW1-8, J2 to J1COL1-8, J3 to J2COL9-16, J4 to J3COL17-24, J5 to J4COL25-32, J6 to J2ROW9-16, J7 to J3ROW17-24, J8 to J4ROW25-32, U1 to U2COL9-16, U2 to U5ROW1-8, U3 to U1COL1-8, U4 to U3COL17-24, U5 to U4COL25-32, U6 to U6ROW9-16, U7 to U7ROW17-24, U8 to U8ROW25-32
Connections:
- net COL_SCLK_IN renamed ROW_SCLK_IN
- net ROW_SLCK_IN renamed COL_SLCK_IN
- net COL_DATA_IN: now also J9.1, U$2.PB4, U1COL1-8.SI; no longer J11.1, U$2.PA11, U5ROW1-8.SI
- net COL_RCLK_IN: now also J10.3, J9.3, U$2.PB5, U1COL1-8.RCK, U2COL9-16.RCK, U3COL17-24.RCK, U4COL25-32.RCK; no longer J11.3, J12.3, U$2.PA9-OSC32OUT, U5ROW1-8.RCK, U6ROW9-16.RCK, U7ROW17-24.RCK, U8ROW25-32.RCK
- net ROW_DATA_IN: now also J11.1, U$2.PA11, U5ROW1-8.SI; no longer J9.1, U$2.PB4, U1COL1-8.SI
- net ROW_RCLK_IN: now also J11.3, J12.3, U$2.PA9-OSC32OUT, U5ROW1-8.RCK, U6ROW9-16.RCK, U7ROW17-24.RCK, U8ROW25-32.RCK; no longer J10.3, J9.3, U$2.PB5, U1COL1-8.RCK, U2COL9-16.RCK, U3COL17-24.RCK, U4COL25-32.RCK

Commit message: Added rx/tx breakout
Parts:
- added J1: 455-1750-1-ND, SparkFun-Connectors:CONN_03
Connections:
- net GND: now also J1.1
- net PA2-U1TX: now also J1.3
- net PA3-U1RX: now also J1.2
Changed lines of the file:
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@@
 <part name="J3ROW17-24" library="SparkFun-Connectors" deviceset="CONN_08" device="&quot;"/>
 <part name="J4ROW25-32" library="SparkFun-Connectors" deviceset="CONN_08" device="&quot;"/>
+<part name="J1" library="SparkFun-Connectors" deviceset="CONN_03" device="" value="455-1750-1-ND"/>
+<part name="GND9" library="supply1" library_urn="urn:adsk.eagle:library:371" deviceset="GND" device=""/>
 </parts>
 <sheets>
@@
 <attribute name="NAME" x="-114.3" y="28.448" size="1.778" layer="95" font="vector"/>
 </instance>
+<instance part="J1" gate="J$1" x="-111.76" y="-50.8" smashed="yes">
+<attribute name="VALUE" x="-114.3" y="-58.166" size="1.778" layer="96" font="vector"/>
+<attribute name="NAME" x="-114.3" y="-45.212" size="1.778" layer="95" font="vector"/>
+</instance>
+<instance part="GND9" gate="1" x="-99.06" y="-63.5" smashed="yes">
+<attribute name="VALUE" x="-101.6" y="-66.04" size="1.778" layer="96"/>
+</instance>
 </instances>
 <busses>
@@
 <pinref part="GND13" gate="1" pin="GND"/>
 </segment>
+<segment>
+<pinref part="J1" gate="J$1" pin="1"/>
+<wire x1="-104.14" y1="-53.34" x2="-99.06" y2="-53.34" width="0.1524" layer="91"/>
+<wire x1="-99.06" y1="-53.34" x2="-99.06" y2="-60.96" width="0.1524" layer="91"/>
+<pinref part="GND9" gate="1" pin="GND"/>
+</segment>
 </net>
 <net name="COL_SLCK_IN" class="0">
@@
 <wire x1="154.94" y1="-20.32" x2="190.5" y2="-20.32" width="0.1524" layer="91"/>
 </segment>
+<segment>
+<pinref part="J1" gate="J$1" pin="3"/>
+<wire x1="-104.14" y1="-48.26" x2="-96.52" y2="-48.26" width="0.1524" layer="91"/>
+<label x="-96.52" y="-48.26" size="1.27" layer="95" xref="yes"/>
+</segment>
 </net>
 <net name="PA3-U1RX" class="0">
@@
 <wire x1="190.5" y1="-12.7" x2="172.72" y2="-12.7" width="0.1524" layer="91"/>
 </segment>
-</net>
+<segment>
+<pinref part="J1" gate="J$1" pin="2"/>
+<wire x1="-104.14" y1="-50.8" x2="-96.52" y2="-50.8" width="0.1524" layer="91"/>
+<label x="-96.52" y="-50.8" size="1.27" layer="95" xref="yes"/>
+</segment>
+</net>
